Commit message: Change collision geometry of wheels to sphere for one point of contact, reducing drift in simulation

File: ros2_packages/av_description/urdf/av.urdf (robot description, URDF)
Before this commit: robot av, 6 links, 5 joints
Links:
- link left_caster_wheel_link: geometry collision sphere radius=0.055; visual cylinder length=0.04 radius=0.05
- link left_wheel_link: geometry collision sphere radius=0.055; visual cylinder length=0.045 radius=0.055
- link right_caster_wheel_link: geometry collision sphere radius=0.055; visual cylinder length=0.04 radius=0.05
- link right_wheel_link: geometry collision sphere radius=0.055; visual cylinder length=0.045 radius=0.055

File: ros2_packages/av_description/urdf/av_core.xacro (robot description, xacro)
@@ -20,5 +20,6 @@
                 <origin xyz="0 0 0" rpy="0 0 0"/>
                 <geometry>
-                    <cylinder radius="${drive_wheel_radius}" length="${drive_wheel_width}"/>
+                    <!-- prevent wheel drift in simulation with a sphere -->
+                    <sphere radius="${drive_wheel_radius}"/>
                 </geometry>
             </collision>

Commit message: Add gazebo launch

File: ros2_packages/av_description/urdf/av.urdf (robot description, URDF)
Before this commit: robot av, 6 links, 5 joints
Links:
- link left_caster_wheel_link: mass 0.32 -> 0.0
- link right_caster_wheel_link: mass 0.32 -> 0.0
Joints:
- joint left_caster_wheel_joint: limit effort=1.0 velocity=10.0 -> effort=100.0 velocity=100.0
- joint left_wheel_joint: limit effort=1.0 velocity=10.0 -> effort=100.0 velocity=100.0
- joint right_caster_wheel_joint: limit effort=1.0 velocity=10.0 -> effort=100.0 velocity=100.0
- joint right_wheel_joint: limit effort=1.0 velocity=10.0 -> effort=100.0 velocity=100.0

File: ros2_packages/av_description/urdf/av.urdf.xacro (robot description, xacro)
@@ -2,3 +2,5 @@
 <robot xmlns:xacro="http://www.ros.org/wiki/xacro" name="av">
     <xacro:include filename="av_core.xacro"/>
+    <xacro:include filename="gazebo.xacro"/>
+    <xacro:include filename="gazebo_control.xacro"/>
 </robot>

File: ros2_packages/av_description/urdf/av_core.xacro (robot description, xacro)
@@ -25,5 +25,5 @@
             </collision>
             <inertial>
-                <mass value="${motor_mass}"/>
+                <mass value="${mass}"/>
                 <inertia
                     ixx="${(mass * ((3 * radius ** 2) + width ** 2)) / 12.0}"
@@ -39,5 +39,5 @@
             <parent link="base_link"/>
             <child link="${prefix}wheel_link"/>
-            <limit velocity="10.0" effort="1.0"/>
+            <limit velocity="100.0" effort="100.0"/>
         </joint>
     </xacro:macro>

Commit message: Stablize gazebo sim, working teleop_twist_keyboard

File: ros2_packages/av_description/urdf/av.urdf (robot description, URDF)
Before this commit: robot av, 6 links, 5 joints
Links:
- link left_caster_wheel_link: mass 0.0 -> 0.1
- link right_caster_wheel_link: mass 0.0 -> 0.1
Joints:
- joint left_caster_wheel_joint: type fixed -> continuous
- joint right_caster_wheel_joint: type fixed -> continuous

File: ros2_packages/av_description/urdf/av_core.xacro (robot description, xacro)
@@ -49,10 +49,10 @@
     <xacro:wheel prefix="right_" reflect="-1.0" type="continuous" radius="${drive_wheel_radius}" width="${drive_wheel_width}" mass="${motor_mass}"/>
     <!-- caster wheels -->
-    <xacro:property name="caster_mass" value="0.0"/>
+    <xacro:property name="caster_mass" value="0.100"/>
     <xacro:property name="caster_wheel_radius" value="${0.10 / 2.0}"/>
     <xacro:property name="caster_wheel_width" value="0.040"/>
     <xacro:property name="caster_x_offset" value="0.45"/>
-    <xacro:wheel prefix="left_caster_" reflect="1.0" type="fixed" radius="${caster_wheel_radius}" width="${caster_wheel_width}" mass="${caster_mass}" x_offset="${caster_x_offset}"/>
-    <xacro:wheel prefix="right_caster_" reflect="-1.0" type="fixed" radius="${caster_wheel_radius}" width="${caster_wheel_width}" mass="${caster_mass}" x_offset="${caster_x_offset}"/>
+    <xacro:wheel prefix="left_caster_" reflect="1.0" type="continuous" radius="${caster_wheel_radius}" width="${caster_wheel_width}" mass="${caster_mass}" x_offset="${caster_x_offset}"/>
+    <xacro:wheel prefix="right_caster_" reflect="-1.0" type="continuous" radius="${caster_wheel_radius}" width="${caster_wheel_width}" mass="${caster_mass}" x_offset="${caster_x_offset}"/>
     <link name="chassis">
         <xacro:property name="body_length" value="0.6"/>

File: ros2_packages/av_description/urdf/gazebo.xacro (robot description, xacro)
@@ -1,5 +1,5 @@
 <?xml version="1.0" encoding="utf-8" ?>
 <robot xmlns:xacro="http://www.ros.org/wiki/xacro" name="av">
-    <xacro:macro name="wheel" params="prefix:='' caster:='false'">
+    <xacro:macro name="wheel" params="prefix:=''">
         <gazebo reference="${prefix}wheel_link">
             <material>Gazebo/Grey</material>
@@ -7,12 +7,7 @@
                 <friction>
                     <ode>
-                        <xacro:if value="${caster == True}">
-                            <mu>0.001</mu>
-                            <mu2>0.001</mu2>
-                        </xacro:if>
-                        <xacro:if value="${caster != True}">
-                            <mu>0.005</mu>
-                            <mu2>0.00005</mu2>
-                        </xacro:if>
+                        <fdir>0 0 1</fdir>
+                        <mu>0.001</mu>
+                        <mu2>0.001</mu2>
                     </ode>
                 </friction>
@@ -23,6 +18,6 @@
     <xacro:wheel prefix="left_"/>
     <xacro:wheel prefix="right_"/>
-    <xacro:wheel prefix="left_caster_" caster="true"/>
-    <xacro:wheel prefix="right_caster_" caster="true"/>
+    <xacro:wheel prefix="left_caster_"/>
+    <xacro:wheel prefix="right_caster_"/>
     <gazebo reference="chassis">
         <material>Gazebo/DarkGrey</material>

Commit message: Refactor and add laser_frame for lidar

File: ros2_packages/av_description/urdf/av.urdf (robot description, URDF)
Before this commit: robot av, 6 links, 5 joints
Links:
- added link laser_frame; collision cylinder length=0.05 radius=0.035; visual cylinder length=0.05 radius=0.035
Joints:
- added joint laser_joint: type fixed, parent chassis, child laser_frame, origin xyz=0.25 0 0.05 rpy=0 0 0

File: ros2_packages/av_description/urdf/av.urdf.xacro (robot description, xacro)
@@ -1,6 +1,6 @@
 <?xml version="1.0" encoding="utf-8" ?>
 <robot xmlns:xacro="http://www.ros.org/wiki/xacro" name="av">
-    <xacro:include filename="av_core.xacro"/>
+    <xacro:include filename="core.xacro"/>
     <xacro:include filename="gazebo.xacro"/>
-    <xacro:include filename="gazebo_control.xacro"/>
+    <xacro:include filename="sensors.xacro"/>
 </robot>

File: ros2_packages/av_description/urdf/core.xacro (robot description, xacro)
@@ -1,4 +1,5 @@
 <?xml version="1.0" encoding="utf-8" ?>
 <robot xmlns:xacro="http://www.ros.org/wiki/xacro" name="av">
+    <xacro:include filename="macros.xacro"/>
     <material name="dark_grey">
         <color rgba="0.2 0.2 0.2 1.0"/>
@@ -24,13 +25,5 @@
                 </geometry>
             </collision>
-            <inertial>
-                <mass value="${mass}"/>
-                <inertia
-                    ixx="${(mass * ((3 * radius ** 2) + width ** 2)) / 12.0}"
-                    iyy="${(mass * ((3 * radius ** 2) + width ** 2)) / 12.0}"
-                    izz="${(mass * radius ** 2) / 2.0}"
-                    ixy="0.0" ixz ="0.0" iyz="0.0"
-                />
-            </inertial>
+            <xacro:cylinder_inertia mass="${mass}" radius="${radius}" width="${width}"/>
         </link>
         <joint name="${prefix}wheel_joint" type="${type}">

File: ros2_packages/av_description/urdf/gazebo.xacro (robot description, xacro)
@@ -23,3 +23,21 @@
         <material>Gazebo/DarkGrey</material>
     </gazebo>
+    <gazebo reference="laser_frame">
+        <material>Gazebo/Black</material>
+    </gazebo>
+    <gazebo>
+        <plugin name='diff_drive' filename='libgazebo_ros_diff_drive.so'>
+            <left_joint>left_wheel_joint</left_joint>
+            <right_joint>right_wheel_joint</right_joint>
+            <wheel_separation>0.29</wheel_separation>
+            <wheel_diameter>0.11</wheel_diameter>
+            <max_wheel_torque>100.0</max_wheel_torque>
+            <max_wheel_acceleration>100.0</max_wheel_acceleration>
+            <odometry_frame>odom</odometry_frame>
+            <robot_base_frame>base_link</robot_base_frame>
+            <publish_odom>true</publish_odom>
+            <publish_odom_tf>true</publish_odom_tf>
+            <publish_wheel_tf>true</publish_wheel_tf>
+        </plugin>
+    </gazebo>
 </robot>

Commit message: Add lidar sensor in gazebo

File: ros2_packages/av_description/urdf/av.urdf (robot description, URDF)
Before this commit: robot av, 7 links, 6 joints
Joints:
- joint laser_joint: origin xyz=0.25 0 0.05 rpy=0 0 0 -> xyz=0.25 0 0.03 rpy=0 0 0

File: ros2_packages/av_description/urdf/gazebo.xacro (robot description, xacro)
@@ -25,4 +25,31 @@
     <gazebo reference="laser_frame">
         <material>Gazebo/Black</material>
+        <sensor name="laser" type="ray">
+            <pose>0 0 0 0 0 0</pose>
+            <visualize>true</visualize>
+            <update_rate>10.0</update_rate>
+            <ray>
+                <scan>
+                    <horizontal>
+                        <samples>720</samples>
+                        <resolution>1</resolution>
+                        <min_angle>-1.5708</min_angle>
+                        <max_angle>1.5708</max_angle>
+                    </horizontal>
+                </scan>
+                <range>
+                    <min>0.1</min>
+                    <max>12</max>
+                    <resolution>0.01</resolution>
+                </range>
+            </ray>
+            <plugin name="laser_controller" filename="libgazebo_ros_ray_sensor.so">
+                <ros>
+                    <argument>~/out:=scan</argument>
+                </ros>
+                <output_type>sensor_msgs/LaserScan</output_type>
+                <frame_name>laser_frame</frame_name>
+            </plugin>
+        </sensor>
     </gazebo>
     <gazebo>

File: ros2_packages/av_description/urdf/sensors.xacro (robot description, xacro)
@@ -25,5 +25,5 @@
     </link>
     <joint name="laser_joint" type="fixed">
-        <origin xyz="0.25 0 ${lidar_height}" rpy="0 0 0"/>
+        <origin xyz="0.25 0 ${0.03}" rpy="0 0 0"/>
         <parent link="chassis"/>
         <child link="laser_frame"/>

Commit message: Add camera_link

File: ros2_packages/av_description/urdf/av.urdf (robot description, URDF)
Before this commit: robot av, 7 links, 6 joints
Links:
- added link camera_link; visual box size=0.025 0.09 0.025
Joints:
- added joint camera_joint: type fixed, parent chassis, child camera_link, origin xyz=-0.05 0 0.15 rpy=0 0 0

File: ros2_packages/av_description/urdf/sensors.xacro (robot description, xacro)
@@ -5,4 +5,5 @@
         <color rgba="0.0 0.0 0.0 1.0"/>
     </material>
+    <!-- lidar -->
     <xacro:property name="lidar_height" value="0.05"/>
     <xacro:property name="lidar_radius" value="${0.07 / 2.0}"/>
@@ -29,3 +30,17 @@
         <child link="laser_frame"/>
     </joint>
+    <!-- camera -->
+    <link name="camera_link" type="fixed">
+        <visual>
+            <geometry>
+                <box size="0.025 0.09 0.025"/>
+            </geometry>
+            <material name="black"/>
+        </visual>
+    </link>
+    <joint name="camera_joint" type="fixed">
+        <origin xyz="-0.05 0 0.15" rpy="0 0 0"/>
+        <parent link="chassis"/>
+        <child link="camera_link"/>
+    </joint>
 </robot>

Commit message: Add camera sensor to gazebo

File: ros2_packages/av_description/urdf/av.urdf (robot description, URDF)
Before this commit: robot av, 8 links, 7 joints
Links:
- added link camera_link_optical
Joints:
- added joint camera_joint_optical: type fixed, parent camera_link, child camera_link_optical, origin xyz=0 0 0 rpy=-1.5707963267948966 0 -1.5707963267948966

File: ros2_packages/av_description/urdf/gazebo.xacro (robot description, xacro)
@@ -23,4 +23,21 @@
         <material>Gazebo/DarkGrey</material>
     </gazebo>
+    <!-- controls -->
+    <gazebo>
+        <plugin name='diff_drive' filename='libgazebo_ros_diff_drive.so'>
+            <left_joint>left_wheel_joint</left_joint>
+            <right_joint>right_wheel_joint</right_joint>
+            <wheel_separation>0.29</wheel_separation>
+            <wheel_diameter>0.11</wheel_diameter>
+            <max_wheel_torque>100.0</max_wheel_torque>
+            <max_wheel_acceleration>100.0</max_wheel_acceleration>
+            <odometry_frame>odom</odometry_frame>
+            <robot_base_frame>base_link</robot_base_frame>
+            <publish_odom>true</publish_odom>
+            <publish_odom_tf>true</publish_odom_tf>
+            <publish_wheel_tf>true</publish_wheel_tf>
+        </plugin>
+    </gazebo>
+    <!-- sensors -->
     <gazebo reference="laser_frame">
         <material>Gazebo/Black</material>
@@ -53,18 +70,28 @@
         </sensor>
     </gazebo>
-    <gazebo>
-        <plugin name='diff_drive' filename='libgazebo_ros_diff_drive.so'>
-            <left_joint>left_wheel_joint</left_joint>
-            <right_joint>right_wheel_joint</right_joint>
-            <wheel_separation>0.29</wheel_separation>
-            <wheel_diameter>0.11</wheel_diameter>
-            <max_wheel_torque>100.0</max_wheel_torque>
-            <max_wheel_acceleration>100.0</max_wheel_acceleration>
-            <odometry_frame>odom</odometry_frame>
-            <robot_base_frame>base_link</robot_base_frame>
-            <publish_odom>true</publish_odom>
-            <publish_odom_tf>true</publish_odom_tf>
-            <publish_wheel_tf>true</publish_wheel_tf>
-        </plugin>
+    <gazebo reference="camera_link">
+        <material>Gazebo/Black</material>
+        <sensor name="camera" type="camera">
+            <pose>0 0 0 0 0 0</pose>
+            <visualize>true</visualize>
+            <update_rate>10.0</update_rate>
+            <!-- RealSense D435i-->
+            <camera>
+                <!-- RGB camera 69 degrees -->
+                <horizontal_fov>1.204</horizontal_fov>
+                <image>
+                    <width>640</width>
+                    <height>480</height>
+                    <format>R8G8B8</format>
+                </image>
+                <clip>
+                    <near>0.05</near>
+                    <far>100.0</far>
+                </clip>
+            </camera>
+            <plugin name="camera_controller" filename="libgazebo_ros_camera.so">
+                <frame_name>camera_link_optical</frame_name>
+            </plugin>
+        </sensor>
     </gazebo>
 </robot>

File: ros2_packages/av_description/urdf/sensors.xacro (robot description, xacro)
@@ -44,3 +44,9 @@
         <child link="camera_link"/>
     </joint>
+    <link name="camera_link_optical"/>
+    <joint name="camera_joint_optical" type="fixed">
+        <origin xyz="0 0 0" rpy="${-pi/2.0} 0 ${-pi/2.0}"/>
+        <parent link="camera_link"/>
+        <child link="camera_link_optical"/>
+    </joint>
 </robot>
