Commit message: Add ros2_control interfaces

File: ros2_packages/av_description/urdf/ros2_control.xacro (robot description, xacro)
@@ -21,4 +21,10 @@
             <state_interface name="position" />
         </joint>
+        <joint name="left_caster_wheel_joint">
+            <state_interface name="position" />
+        </joint>
+        <joint name="right_caster_wheel_joint">
+            <state_interface name="position" />
+        </joint>
     </ros2_control>
     <gazebo>
