Commit message: Refactor wheel macro

File: ros2_packages/av_description/urdf/core.xacro (robot description, xacro)
@@ -9,5 +9,5 @@
     </material>
     <xacro:property name="y_wheel_offset" value="${0.29 / 2.0}"/>
-    <xacro:macro name="wheel" params="prefix:='' reflect:=1.0 type radius width mass x_offset:='0'">
+    <xacro:macro name="wheel" params="prefix:='' reflect:=1.0 radius width mass x_offset:='0'">
         <link name="${prefix}wheel_link">
             <visual>
@@ -27,5 +27,5 @@
             <xacro:cylinder_inertia mass="${mass}" radius="${radius}" width="${width}"/>
         </link>
-        <joint name="${prefix}wheel_joint" type="${type}">
+        <joint name="${prefix}wheel_joint" type="continuous">
             <axis xyz="0 0 1"/>
             <origin xyz="${x_offset} ${reflect * y_wheel_offset} ${radius}" rpy="${-pi / 2.0} 0 0"/>
@@ -39,6 +39,6 @@
     <xacro:property name="drive_wheel_radius" value="${0.11 / 2.0}"/>
     <xacro:property name="drive_wheel_width" value="0.045"/>
-    <xacro:wheel prefix="left_" reflect="1.0" type="continuous" radius="${drive_wheel_radius}" width="${drive_wheel_width}" mass="${motor_mass}"/>
-    <xacro:wheel prefix="right_" reflect="-1.0" type="continuous" radius="${drive_wheel_radius}" width="${drive_wheel_width}" mass="${motor_mass}"/>
+    <xacro:wheel prefix="left_" reflect="1.0" radius="${drive_wheel_radius}" width="${drive_wheel_width}" mass="${motor_mass}"/>
+    <xacro:wheel prefix="right_" reflect="-1.0" radius="${drive_wheel_radius}" width="${drive_wheel_width}" mass="${motor_mass}"/>
     <!-- caster wheels -->
     <xacro:property name="caster_mass" value="0.100"/>
@@ -46,6 +46,6 @@
     <xacro:property name="caster_wheel_width" value="0.040"/>
     <xacro:property name="caster_x_offset" value="0.45"/>
-    <xacro:wheel prefix="left_caster_" reflect="1.0" type="continuous" radius="${caster_wheel_radius}" width="${caster_wheel_width}" mass="${caster_mass}" x_offset="${caster_x_offset}"/>
-    <xacro:wheel prefix="right_caster_" reflect="-1.0" type="continuous" radius="${caster_wheel_radius}" width="${caster_wheel_width}" mass="${caster_mass}" x_offset="${caster_x_offset}"/>
+    <xacro:wheel prefix="left_caster_" reflect="1.0" radius="${caster_wheel_radius}" width="${caster_wheel_width}" mass="${caster_mass}" x_offset="${caster_x_offset}"/>
+    <xacro:wheel prefix="right_caster_" reflect="-1.0" radius="${caster_wheel_radius}" width="${caster_wheel_width}" mass="${caster_mass}" x_offset="${caster_x_offset}"/>
     <link name="chassis">
         <xacro:property name="body_length" value="0.6"/>

Commit message: Update wheel masses from real measurements

File: ros2_packages/av_description/urdf/core.xacro (robot description, xacro)
@@ -36,11 +36,11 @@
     </xacro:macro>
     <!-- drive wheels -->
-    <xacro:property name="motor_mass" value="0.320"/>
+    <xacro:property name="drive_wheel_mass" value="0.322"/>
     <xacro:property name="drive_wheel_radius" value="${0.11 / 2.0}"/>
     <xacro:property name="drive_wheel_width" value="0.045"/>
-    <xacro:wheel prefix="left_" reflect="1.0" radius="${drive_wheel_radius}" width="${drive_wheel_width}" mass="${motor_mass}"/>
-    <xacro:wheel prefix="right_" reflect="-1.0" radius="${drive_wheel_radius}" width="${drive_wheel_width}" mass="${motor_mass}"/>
+    <xacro:wheel prefix="left_" reflect="1.0" radius="${drive_wheel_radius}" width="${drive_wheel_width}" mass="${drive_wheel_mass}"/>
+    <xacro:wheel prefix="right_" reflect="-1.0" radius="${drive_wheel_radius}" width="${drive_wheel_width}" mass="${drive_wheel_mass}"/>
     <!-- caster wheels -->
-    <xacro:property name="caster_mass" value="0.100"/>
+    <xacro:property name="caster_mass" value="0.260"/>
     <xacro:property name="caster_wheel_radius" value="${0.10 / 2.0}"/>
     <xacro:property name="caster_wheel_width" value="0.040"/>
