Commit message: Add working ros2_control av_bringup

File: av_description/urdf/ros2_control.xacro (robot description, xacro)
@@ -1,12 +1,16 @@
 <?xml version="1.0" encoding="utf-8" ?>
 <robot xmlns:xacro="http://www.ros.org/wiki/xacro" name="av">
-    <ros2_control name="GazeboSystem" type="system">
+    <ros2_control name="DriveWheels" type="actuator">
         <hardware>
-            <plugin>gazebo_ros2_control/GazeboSystem</plugin>
+            <!-- <plugin>gazebo_ros2_control/GazeboSystem</plugin> -->
+            <plugin>av_hardware/AvHardwareInterface</plugin>
         </hardware>
         <joint name="left_wheel_joint">
+            <command_interface name="position">
+                <param name="initial_value">0.0</param>
+            </command_interface>
             <command_interface name="velocity">
-                <param name="min">-10</param>
-                <param name="max">10</param>
+                <param name="min">-10.0</param>
+                <param name="max">10.0</param>
             </command_interface>
             <state_interface name="position" />
@@ -14,22 +18,25 @@
         </joint>
         <joint name="right_wheel_joint">
+            <command_interface name="position">
+                <param name="initial_value">0.0</param>
+            </command_interface>
             <command_interface name="velocity">
-                <param name="min">-10</param>
-                <param name="max">10</param>
+                <param name="min">-10.0</param>
+                <param name="max">10.0</param>
             </command_interface>
             <state_interface name="velocity" />
             <state_interface name="position" />
         </joint>
-        <joint name="left_caster_wheel_joint">
+        <!-- <joint name="left_caster_wheel_joint">
             <state_interface name="position" />
         </joint>
         <joint name="right_caster_wheel_joint">
             <state_interface name="position" />
-        </joint>
+        </joint> -->
     </ros2_control>
-    <gazebo>
+    <!-- <gazebo>
         <plugin filename="libgazebo_ros2_control.so" name="gazebo_ros2_control">
             <parameters>$(find av_description)/config/controllers.yaml</parameters>
         </plugin>
-    </gazebo>
+    </gazebo> -->
 </robot>

File: av_description/urdf/sensors.xacro (robot description, xacro)
@@ -11,4 +11,5 @@
     <link name="laser_frame">
         <visual>
+            <origin xyz="0 0 0" rpy="0 0 ${pi}"/>
             <geometry>
                 <cylinder radius="${lidar_radius}" length="${lidar_height}"/>
@@ -38,4 +39,9 @@
             <material name="black"/>
         </visual>
+        <collision>
+            <geometry>
+                <box size="0.025 0.09 0.025"/>
+            </geometry>
+        </collision>
     </link>
     <joint name="camera_joint" type="fixed">
