Commit message: Restore gazebo

File: av_description/urdf/av.urdf.xacro (robot description, xacro)
@@ -1,7 +1,14 @@
 <?xml version="1.0" encoding="utf-8" ?>
 <robot xmlns:xacro="http://www.ros.org/wiki/xacro" name="av">
+    <xacro:arg name="use_ros2_control" default="true"/>
+    <xacro:arg name="sim_mode" default="false"/>
     <xacro:include filename="core.xacro"/>
     <xacro:include filename="gazebo.xacro"/>
     <xacro:include filename="sensors.xacro"/>
-    <xacro:include filename="ros2_control.xacro"/>
+    <xacro:if value="$(arg use_ros2_control)">
+        <xacro:include filename="ros2_control.xacro"/>
+    </xacro:if>
+    <xacro:if value="$(arg sim_mode)">
+        <xacro:include filename="gazebo_control.xacro"/>
+    </xacro:if>
 </robot>

File: av_description/urdf/gazebo.xacro (robot description, xacro)
@@ -4,8 +4,4 @@
         <gazebo reference="${prefix}wheel_link">
             <material>Gazebo/Grey</material>
-            <!-- <surface>
-                <friction>
-                    <ode> -->
-                        <!-- <fdir>0 0 1</fdir> -->
         <xacro:if value="${caster}">
             <mu1 value="0.000001"/>

File: av_description/urdf/ros2_control.xacro (robot description, xacro)
@@ -1,8 +1,12 @@
 <?xml version="1.0" encoding="utf-8" ?>
-<robot xmlns:xacro="http://www.ros.org/wiki/xacro" name="av">
+<robot xmlns:xacro="http://www.ros.org/wiki/xacro" name="av" >
     <ros2_control name="DriveWheels" type="actuator">
         <hardware>
-            <!-- <plugin>gazebo_ros2_control/GazeboSystem</plugin> -->
-            <plugin>av_hardware/AvHardwareInterface</plugin>
+            <xacro:unless value="$(arg sim_mode)">
+                <plugin>av_hardware/AvHardwareInterface</plugin>
+            </xacro:unless>
+            <xacro:if value="$(arg sim_mode)">
+                <plugin>gazebo_ros2_control/GazeboSystem</plugin>
+            </xacro:if>
         </hardware>
         <joint name="left_wheel_joint">
@@ -11,6 +15,6 @@
             </command_interface>
             <command_interface name="velocity">
-                <param name="min">-10.0</param>
-                <param name="max">10.0</param>
+                <param name="min">-5.0</param>
+                <param name="max">5.0</param>
             </command_interface>
             <state_interface name="position" />
@@ -22,21 +26,17 @@
             </command_interface>
             <command_interface name="velocity">
-                <param name="min">-10.0</param>
-                <param name="max">10.0</param>
+                <param name="min">-5.0</param>
+                <param name="max">5.0</param>
             </command_interface>
             <state_interface name="velocity" />
             <state_interface name="position" />
         </joint>
-        <!-- <joint name="left_caster_wheel_joint">
-            <state_interface name="position" />
-        </joint>
-        <joint name="right_caster_wheel_joint">
-            <state_interface name="position" />
-        </joint> -->
     </ros2_control>
-    <!-- <gazebo>
-        <plugin filename="libgazebo_ros2_control.so" name="gazebo_ros2_control">
-            <parameters>$(find av_description)/config/controllers.yaml</parameters>
-        </plugin>
-    </gazebo> -->
+    <xacro:if value="$(arg sim_mode)">
+        <gazebo>
+            <plugin filename="libgazebo_ros2_control.so" name="gazebo_ros2_control">
+                <parameters>$(find av_description)/config/controllers.yaml</parameters>
+            </plugin>
+        </gazebo>
+    </xacro:if>
 </robot>
