Commit message: Add base_footprint

File: av_description/urdf/core.xacro (robot description, xacro)
@@ -84,3 +84,9 @@
     </joint>
     <link name="base_link"/>
+    <joint name="base_footprint_joint" type="fixed">
+        <origin xyz="0 0 0" rpy="0 0 0"/>
+        <parent link="base_link"/>
+        <child link="base_footprint"/>
+    </joint>
+    <link name="base_footprint"/>
 </robot>
