Commit message: Rotate LiDAR 180

File: av_description/urdf/sensors.xacro (robot description, xacro)
@@ -27,5 +27,5 @@
     </link>
     <joint name="laser_joint" type="fixed">
-        <origin xyz="0.25 0 ${0.03}" rpy="0 0 0"/>
+        <origin xyz="0.25 0 ${0.03}" rpy="0 0 ${pi}"/>
         <parent link="chassis"/>
         <child link="laser_frame"/>

Commit message: Add realsense to urdf

File: av_description/urdf/sensors.xacro (robot description, xacro)
@@ -32,27 +32,36 @@
     </joint>
     <!-- camera -->
-    <link name="camera_link" type="fixed">
-        <visual>
-            <geometry>
-                <box size="0.025 0.09 0.025"/>
-            </geometry>
-            <material name="black"/>
-        </visual>
-        <collision>
-            <geometry>
-                <box size="0.025 0.09 0.025"/>
-            </geometry>
-        </collision>
-    </link>
-    <joint name="camera_joint" type="fixed">
-        <origin xyz="-0.05 0 0.15" rpy="0 0 0"/>
-        <parent link="chassis"/>
-        <child link="camera_link"/>
-    </joint>
-    <link name="camera_link_optical"/>
-    <joint name="camera_joint_optical" type="fixed">
-        <origin xyz="0 0 0" rpy="${-pi/2.0} 0 ${-pi/2.0}"/>
-        <parent link="camera_link"/>
-        <child link="camera_link_optical"/>
-    </joint>
+    <xacro:property name="use_realsense" value="true"/>
+    <xacro:if value="${use_realsense}">
+        <xacro:include filename="$(find realsense2_description)/urdf/_d455.urdf.xacro"/>
+        <xacro:sensor_d455 parent="chassis" use_nominal_extrinsics="true">
+            <origin xyz="-0.05 0 0.15" rpy="0 0 0"/>
+        </xacro:sensor_d455>
+    </xacro:if>
+    <xacro:unless value="${use_realsense}">
+        <joint name="camera_joint" type="fixed">
+            <origin xyz="-0.05 0 0.15" rpy="0 0 0"/>
+            <parent link="chassis"/>
+            <child link="camera_link"/>
+        </joint>
+        <link name="camera_link" type="fixed">
+            <visual>
+                <geometry>
+                    <box size="0.025 0.09 0.025"/>
+                </geometry>
+                <material name="black"/>
+            </visual>
+            <collision>
+                <geometry>
+                    <box size="0.025 0.09 0.025"/>
+                </geometry>
+            </collision>
+        </link>
+        <link name="camera_link_optical"/>
+        <joint name="camera_joint_optical" type="fixed">
+            <origin xyz="0 0 0" rpy="${-pi/2.0} 0 ${-pi/2.0}"/>
+            <parent link="camera_link"/>
+            <child link="camera_link_optical"/>
+        </joint>
+    </xacro:unless>
 </robot>
